Commit message: rmrc and asc working + jla + sca

File: planar_bot_description/urdf/planar_bot.xacro (robot description, xacro)
@@ -134,5 +134,5 @@
     </inertial>
   </link>
-  <joint name="joint1" type="continuous">
+  <joint name="joint1" type="revolute">
     <parent link="base_link"/>
     <child link="link1"/>
@@ -140,6 +140,7 @@
     <axis xyz="0 0 1"/>
     <dynamics damping="0.7"/>
-  </joint>
-  <joint name="joint2" type="continuous">
+    <limit effort="80" velocity="8.0" lower="-3.0" upper="3.0" />
+  </joint>
+  <joint name="joint2" type="revolute">
     <parent link="link1"/>
     <child link="link2"/>
@@ -147,6 +148,7 @@
     <axis xyz="0 0 1"/>
     <dynamics damping="0.7"/>
-  </joint>
-  <joint name="joint3" type="continuous">
+    <limit effort="80" velocity="8.0" lower="-3.0" upper="3.0" />
+  </joint>
+  <joint name="joint3" type="revolute">
     <parent link="link2"/>
     <child link="link3"/>
@@ -154,6 +156,7 @@
     <axis xyz="0 0 1"/>
     <dynamics damping="0.7"/>
-  </joint>
-  <joint name="joint4" type="continuous">
+    <limit effort="80" velocity="8.0" lower="-3.0" upper="3.0" />
+  </joint>
+  <joint name="joint4" type="revolute">
     <parent link="link3"/>
     <child link="link4"/>
@@ -161,4 +164,5 @@
     <axis xyz="0 0 1"/>
     <dynamics damping="0.7"/>
+    <limit effort="80" velocity="8.0" lower="-3.0" upper="3.0" />
   </joint>
   <transmission name="tran1">

Commit message: finished test setup

File: planar_bot_description/urdf/planar_bot.xacro (robot description, xacro)
@@ -140,5 +140,5 @@
     <axis xyz="0 0 1"/>
     <dynamics damping="0.7"/>
-    <limit effort="80" velocity="8.0" lower="-3.0" upper="3.0" />
+    <limit effort="80" velocity="8.0" lower="-0.3" upper="3.45" />
   </joint>
   <joint name="joint2" type="revolute">
